File: HW/ps002.sch (KiCad schematic (older format))
At the start: 17 parts, among them U1 MC34063

Commit message: Schematic diagram completted PCB design started
Parts:
- added J1: USB, USB_B, symbol USB
- added J2: OUT, HDR-3, symbol CONN_3
- C1, C3, C4, C5, C6, C7: footprint ~ -> C2P_D4
- C2: footprint ~ -> C1
- D1, D2, D3: footprint ~ -> D4
- L1: footprint ~ -> L2_D3.5
- L2, L3, R1: footprint ~ -> R5
- R2, R3: footprint ~ -> R4
- U1: footprint (none) -> DIP-8
Connections:
- net labels added: VCC
- wire segments 37 -> 43
Changed lines of the file:
@@
 LIBS:contrib
 LIBS:valves
+LIBS:ps002-cache
 EELAYER 27 0
 EELAYER END
@@
 Sheet 1 1
 Title ""
-Date "16 sep 2014"
+Date "18 sep 2014"
 Rev ""
 Comp ""
@@
 F 0 "U1" H 5150 3100 60  0000 C CNN
 F 1 "MC34063" H 5300 3600 60  0000 C CNN
-F 2 "" H 5200 3350 60  0000 C CNN
+F 2 "DIP-8" H 5200 3350 60  0001 C CNN
 F 3 "" H 5200 3350 60  0000 C CNN
 	1    5350 3350
@@
 F 0 "C1" H 4450 3400 40  0000 C CNN
 F 1 "470uF/10V" H 4500 3700 40  0000 C CNN
-F 2 "~" H 4450 3550 60  0000 C CNN
+F 2 "C2P_D4" H 4450 3550 60  0001 C CNN
 F 3 "~" H 4450 3550 60  0000 C CNN
 	1    4450 3550
@@
 F 0 "R1" H 4650 3225 40  0000 C CNN
 F 1 "R47/1W" H 4650 3375 40  0000 C CNN
-F 2 "~" H 4650 3300 60  0000 C CNN
+F 2 "R5" H 4650 3300 60  0001 C CNN
 F 3 "~" H 4650 3300 60  0000 C CNN
 	1    4650 3300
@@
 F 0 "L1" H 5350 2900 60  0000 C CNN
 F 1 "100uH" H 5350 3050 60  0000 C CNN
-F 2 "~" H 5350 2950 60  0000 C CNN
+F 2 "L2_D3.5" H 5350 2950 60  0001 C CNN
 F 3 "~" H 5350 2950 60  0000 C CNN
 	1    5350 2950
@@
 F 0 "C2" H 5850 3500 40  0000 C CNN
 F 1 "330pF" H 5850 3800 40  0000 C CNN
-F 2 "~" H 5850 3650 60  0000 C CNN
+F 2 "C1" H 5850 3650 60  0001 C CNN
 F 3 "~" H 5850 3650 60  0000 C CNN
 	1    5850 3650
@@
 $EndComp
 $Comp
-L GND #PWR3
+L GND #PWR01
 U 1 1 54189ED5
 P 5850 3800
-F 0 "#PWR3" H 5850 3800 30  0001 C CNN
+F 0 "#PWR01" H 5850 3800 30  0001 C CNN
 F 1 "GND" H 5850 3730 30  0001 C CNN
 F 2 "" H 5850 3800 60  0000 C CNN
@@
 F 0 "C4" H 6825 3150 40  0000 C CNN
 F 1 "470uF/25V" V 6875 3500 40  0000 C CNN
-F 2 "~" H 6800 3300 60  0000 C CNN
+F 2 "C2P_D4" H 6800 3300 60  0001 C CNN
 F 3 "~" H 6800 3300 60  0000 C CNN
 	1    6800 3300
@@
 F 0 "C5" H 6825 3400 40  0000 C CNN
 F 1 "470uF/25V" V 6875 3725 40  0000 C CNN
-F 2 "~" H 6800 3550 60  0000 C CNN
+F 2 "C2P_D4" H 6800 3550 60  0001 C CNN
 F 3 "~" H 6800 3550 60  0000 C CNN
 	1    6800 3550
@@
 F 0 "L2" H 7200 3150 60  0000 C CNN
 F 1 "1uH" H 7200 3300 60  0000 C CNN
-F 2 "~" H 7200 3200 60  0000 C CNN
+F 2 "R5" H 7200 3200 60  0001 C CNN
 F 3 "~" H 7200 3200 60  0000 C CNN
 	1    7200 3200
@@
 F 0 "L3" H 7200 3600 60  0000 C CNN
 F 1 "1uH" H 7200 3750 60  0000 C CNN
-F 2 "~" H 7200 3650 60  0000 C CNN
+F 2 "R5" H 7200 3650 60  0001 C CNN
 F 3 "~" H 7200 3650 60  0000 C CNN
 	1    7200 3650
@@
 F 0 "C6" H 7600 3150 40  0000 C CNN
 F 1 "470uF/16V" V 7675 3500 40  0000 C CNN
-F 2 "~" H 7600 3300 60  0000 C CNN
+F 2 "C2P_D4" H 7600 3300 60  0001 C CNN
 F 3 "~" H 7600 3300 60  0000 C CNN
 	1    7600 3300
@@
 F 0 "C7" H 7600 3400 40  0000 C CNN
 F 1 "470uF/16V" V 7675 3750 40  0000 C CNN
-F 2 "~" H 7600 3550 60  0000 C CNN
+F 2 "C2P_D4" H 7600 3550 60  0001 C CNN
 F 3 "~" H 7600 3550 60  0000 C CNN
 	1    7600 3550
@@
 F 0 "D1" H 6375 3225 40  0000 C CNN
 F 1 "1N5819" H 6675 3150 40  0000 C CNN
-F 2 "~" H 6500 3200 60  0000 C CNN
+F 2 "D4" H 6500 3200 60  0001 C CNN
 F 3 "~" H 6500 3200 60  0000 C CNN
 	1    6500 3200
@@
 F 0 "D3" H 6625 3600 40  0000 C CNN
 F 1 "1N5819" H 6325 3700 40  0000 C CNN
-F 2 "~" H 6500 3650 60  0000 C CNN
+F 2 "D4" H 6500 3650 60  0001 C CNN
 F 3 "~" H 6500 3650 60  0000 C CNN
 	1    6500 3650
@@
 F 0 "C3" H 6250 3475 40  0000 C CNN
 F 1 "470uF/25V" H 6475 3275 40  0000 C CNN
-F 2 "~" H 6250 3325 60  0000 C CNN
+F 2 "C2P_D4" H 6250 3325 60  0001 C CNN
 F 3 "~" H 6250 3325 60  0000 C CNN
 	1    6250 3325
@@
 F 0 "D2" H 6375 3450 40  0000 C CNN
 F 1 "1N5819" H 6675 3375 40  0000 C CNN
-F 2 "~" H 6500 3425 60  0000 C CNN
+F 2 "D4" H 6500 3425 60  0001 C CNN
 F 3 "~" H 6500 3425 60  0000 C CNN
 	1    6500 3425
@@
 F 0 "R3" H 6500 2875 40  0000 C CNN
 F 1 "13K" H 6500 3025 40  0000 C CNN
-F 2 "~" H 6500 2950 60  0000 C CNN
+F 2 "R4" H 6500 2950 60  0001 C CNN
 F 3 "~" H 6500 2950 60  0000 C CNN
 	1    6500 2950
@@
 F 0 "R2" H 4900 3825 40  0000 C CNN
 F 1 "1K5" H 4900 3975 40  0000 C CNN
-F 2 "~" H 4900 3900 60  0000 C CNN
+F 2 "R4" H 4900 3900 60  0001 C CNN
 F 3 "~" H 4900 3900 60  0000 C CNN
 	1    4900 3900
@@
 $EndComp
 Wire Wire Line
-	6700 3425 7850 3425
+	6700 3425 8300 3425
 Wire Wire Line
 	7600 3400 7600 3450
@@
 Connection ~ 6800 3650
 Wire Wire Line
-	7400 3650 7600 3650
+	7400 3650 8300 3650
 Wire Wire Line
 	6700 3200 7000 3200
 Connection ~ 6800 3200
 Wire Wire Line
-	7400 3200 7600 3200
+	7400 3200 8300 3200
 Wire Wire Line
 	6700 2950 6800 2950
@@
 	6250 3425 6300 3425
 $Comp
-L GND #PWR4
+L GND #PWR02
 U 1 1 5418A239
 P 7850 3500
-F 0 "#PWR4" H 7850 3500 30  0001 C CNN
+F 0 "#PWR02" H 7850 3500 30  0001 C CNN
 F 1 "GND" H 7850 3430 30  0001 C CNN
 F 2 "" H 7850 3500 60  0000 C CNN
@@
 	4900 3700 4900 3500
 $Comp
-L GND #PWR2
+L GND #PWR03
 U 1 1 5418A2A6
 P 4900 4150
-F 0 "#PWR2" H 4900 4150 30  0001 C CNN
+F 0 "#PWR03" H 4900 4150 30  0001 C CNN
 F 1 "GND" H 4900 4080 30  0001 C CNN
 F 2 "" H 4900 4150 60  0000 C CNN
@@
 	5800 2950 5800 3200
 Wire Wire Line
-	4450 3300 4450 3450
+	4450 3150 4450 3450
 Wire Wire Line
 	4900 3400 4450 3400
 Connection ~ 4450 3400
 $Comp
-L GND #PWR1
+L GND #PWR04
 U 1 1 5418A3C4
 P 4450 3700
-F 0 "#PWR1" H 4450 3700 30  0001 C CNN
+F 0 "#PWR04" H 4450 3700 30  0001 C CNN
 F 1 "GND" H 4450 3630 30  0001 C CNN
 F 2 "" H 4450 3700 60  0000 C CNN
@@
 Wire Wire Line
 	4450 3650 4450 3700
+$Comp
+L USB J1
+U 1 1 541A543A
+P 3650 3050
+F 0 "J1" H 3600 3450 60  0000 C CNN
+F 1 "USB" V 3400 3200 60  0000 C CNN
+F 2 "USB_B" H 3650 3050 60  0001 C CNN
+F 3 "" H 3650 3050 60  0000 C CNN
+	1    3650 3050
+	1    0    0    -1
+$EndComp
+$Comp
+L GND #PWR05
+U 1 1 541A54B8
+P 3150 3650
+F 0 "#PWR05" H 3150 3650 30  0001 C CNN
+F 1 "GND" H 3150 3580 30  0001 C CNN
+F 2 "" H 3150 3650 60  0000 C CNN
+F 3 "" H 3150 3650 60  0000 C CNN
+	1    3150 3650
+	1    0    0    -1
+$EndComp
+Wire Wire Line
+	3250 3400 3150 3400
+Wire Wire Line
+	3150 3400 3150 3650
+$Comp
+L VCC #PWR06
+U 1 1 541A54F5
+P 3150 3200
+F 0 "#PWR06" H 3150 3300 30  0001 C CNN
+F 1 "VCC" H 3150 3300 30  0000 C CNN
+F 2 "" H 3150 3200 60  0000 C CNN
+F 3 "" H 3150 3200 60  0000 C CNN
+	1    3150 3200
+	1    0    0    -1
+$EndComp
+Wire Wire Line
+	3250 3250 3150 3250
+Wire Wire Line
+	3150 3250 3150 3200
+$Comp
+L VCC #PWR07
+U 1 1 541A5535
+P 4450 3150
+F 0 "#PWR07" H 4450 3250 30  0001 C CNN
+F 1 "VCC" H 4450 3250 30  0000 C CNN
+F 2 "" H 4450 3150 60  0000 C CNN
+F 3 "" H 4450 3150 60  0000 C CNN
+	1    4450 3150
+	1    0    0    -1
+$EndComp
+Connection ~ 4450 3300
+$Comp
+L CONN_3 J2
+U 1 1 541A55A9
+P 8650 3425
+F 0 "J2" V 8600 3425 50  0000 C CNN
+F 1 "OUT" V 8700 3425 40  0000 C CNN
+F 2 "HDR-3" H 8650 3425 60  0001 C CNN
+F 3 "" H 8650 3425 60  0000 C CNN
+	1    8650 3425
+	1    0    0    -1
+$EndComp
+Wire Wire Line
+	8300 3200 8300 3325
+Connection ~ 7600 3200
+Wire Wire Line
+	8300 3650 8300 3525
+Connection ~ 7600 3650
+Connection ~ 7850 3425
 $EndSCHEMATC

Commit message: PS002 B version added Separate controllers for positive and negative sides
Parts:
- J1: footprint USB_B -> USB-B
Changed lines of the file:
@@
 F 0 "J1" H 3600 3450 60  0000 C CNN
 F 1 "USB" V 3400 3200 60  0000 C CNN
-F 2 "USB_B" H 3650 3050 60  0001 C CNN
+F 2 "USB-B" H 3650 3050 60  0001 C CNN
 F 3 "" H 3650 3050 60  0000 C CNN
 	1    3650 3050

Commit message: Update cache
Parts:
- U1: symbol MC34063 -> MC34063-RESCUE-ps002
Changed lines of the file:
@@
 EESchema Schematic File Version 2
+LIBS:ps002-rescue
 LIBS:suf
 LIBS:conn
@@
 LIBS:memory
 LIBS:xilinx
-LIBS:special
 LIBS:microcontrollers
 LIBS:dsp
@@
 LIBS:valves
 LIBS:ps002-cache
-EELAYER 27 0
+EELAYER 25 0
 EELAYER END
 $Descr A4 11693 8268
@@
 $EndDescr
 $Comp
-L MC34063 U1
+L MC34063-RESCUE-ps002 U1
 U 1 1 54189DB0
 P 5350 3350
@@
 $EndComp
 $Comp
-L GND #PWR01
+L GND-RESCUE-ps002 #PWR01
 U 1 1 54189ED5
 P 5850 3800
@@
 	6250 3425 6300 3425
 $Comp
-L GND #PWR02
+L GND-RESCUE-ps002 #PWR02
 U 1 1 5418A239
 P 7850 3500
@@
 	4900 3700 4900 3500
 $Comp
-L GND #PWR03
+L GND-RESCUE-ps002 #PWR03
 U 1 1 5418A2A6
 P 4900 4150
@@
 Connection ~ 4450 3400
 $Comp
-L GND #PWR04
+L GND-RESCUE-ps002 #PWR04
 U 1 1 5418A3C4
 P 4450 3700
@@
 $EndComp
 $Comp
-L GND #PWR05
+L GND-RESCUE-ps002 #PWR05
 U 1 1 541A54B8
 P 3150 3650
