File: HW/ps002b.sch (KiCad schematic (older format))
At the start: 24 parts, among them J1 USB, J2 OUT, U1 MC34063, U2 MC34063

Commit message: Update cache
Parts:
- U1, U2: symbol MC34063 -> MC34063-RESCUE-ps002b
Changed lines of the file:
@@
 EESchema Schematic File Version 2
+LIBS:ps002b-rescue
 LIBS:suf
 LIBS:conn
@@
 LIBS:memory
 LIBS:xilinx
-LIBS:special
 LIBS:microcontrollers
 LIBS:dsp
@@
 LIBS:contrib
 LIBS:valves
-EELAYER 27 0
+LIBS:ps002b-cache
+EELAYER 25 0
 EELAYER END
 $Descr A4 11693 8268
@@
 $EndDescr
 $Comp
-L MC34063 U1
+L MC34063-RESCUE-ps002b U1
 U 1 1 54189DB0
 P 5350 3350
@@
 $EndComp
 $Comp
-L GND #PWR01
+L GND-RESCUE-ps002b #PWR01
 U 1 1 54189ED5
 P 5850 3800
@@
 	6250 4650 6250 4750
 $Comp
-L GND #PWR02
+L GND-RESCUE-ps002b #PWR02
 U 1 1 5418A239
 P 7800 4500
@@
 	4900 3700 4900 3500
 $Comp
-L GND #PWR03
+L GND-RESCUE-ps002b #PWR03
 U 1 1 5418A2A6
 P 4900 4150
@@
 Connection ~ 4050 3400
 $Comp
-L GND #PWR04
+L GND-RESCUE-ps002b #PWR04
 U 1 1 5418A3C4
 P 4050 3700
@@
 $EndComp
 $Comp
-L GND #PWR05
+L GND-RESCUE-ps002b #PWR05
 U 1 1 541A54B8
 P 3350 4900
@@
 Connection ~ 7800 4425
 $Comp
-L MC34063 U2
+L MC34063-RESCUE-ps002b U2
 U 1 1 54207458
 P 5350 4700
@@
 $EndComp
 $Comp
-L GND #PWR08
+L GND-RESCUE-ps002b #PWR08
 U 1 1 54207476
 P 6250 5300
@@
 	4900 5050 4900 4850
 $Comp
-L GND #PWR09
+L GND-RESCUE-ps002b #PWR09
 U 1 1 542074EC
 P 4900 5500
